Commit message: Camera added to the top of the arena.

File: src/bot_gazebo/urdf/camera_old.urdf.xacro (robot description, xacro)
@@ -1,4 +1,10 @@
-<?xml version="1.0" encoding="utf-8"?>
-<robot name="camera">
+<?xml version="1.0"?>
+<robot name="arena_cam" xmlns:xacro="http://www.ros.org/wiki/xacro">
+  <xacro:macro name="arena_cam">
+  <joint name="camera_joint" type="fixed">
+    <parent link="world"/>
+    <child link="camera_link"/>
+    <origin xyz="0 0 5" rpy="0 0 0"/>
+  </joint>
   <link name="camera_link">
     <inertial>
@@ -25,9 +31,4 @@
     </visual>
   </link>
-  <joint name="camera_joint" type="fixed">
-    <parent link="world"/>
-    <child link="camera_link"/>
-    <origin xyz="0 0 5" rpy="0 0 0"/>
-  </joint>
   <gazebo reference="camera_link">
     <sensor type="camera" name="camera_sensor">
@@ -46,5 +47,5 @@
         </clip>
       </camera>
-      <plugin name="camera_camera_controller" filename="libgazebo_ros_camera.so">
+      <plugin name="camera_controller" filename="libgazebo_ros_camera.so">
         <alwaysOn>true</alwaysOn>
         <updateRate>0.0</updateRate>
@@ -62,3 +63,5 @@
     </sensor>
   </gazebo>
+  </xacro:macro>
+  <xacro:arena_cam/>
 </robot>
