Commit message: arena

File: src/bot_description/urdf/base/bot_base.urdf.xacro (robot description, xacro)
@@ -21,5 +21,5 @@
   <link name="base_link">
     <inertial>
-      <mass value="125.0" />
+      <mass value="12.50" />
       <origin xyz="0 0 0" />
       <inertia  ixx="1.391" ixy="0.004"  ixz="0.0"  iyy="6.853"  iyz="0.0"  izz="6.125" />

Commit message: Map has been aligned perfectly.
Bot size has been scaled (2X) as its size feel too small when compared
to whole arena space.
camera parameter hxw updated to have 500 as its value
map_create node updated.

File: src/bot_description/urdf/base/bot_base.urdf.xacro (robot description, xacro)
@@ -28,5 +28,5 @@
        <origin xyz="0 0.02 0" rpy="0 0 3.14" />
        <geometry>
-	     <mesh filename="package://bot_description/meshes/base/custom_base.dae"/>
+	     <mesh filename="package://bot_description/meshes/base/custom_base_scaled.dae"/>
        </geometry>
        <material name="darkgrey">
@@ -37,5 +37,5 @@
        <origin xyz="0 0.02 0" rpy="0 0 3.14" />
        <geometry>
-         <mesh filename="package://bot_description/meshes/base/custom_base.dae"/>
+         <mesh filename="package://bot_description/meshes/base/custom_base_scaled.dae"/>
        </geometry>
     </collision>

File: src/bot_description/urdf/full/bot.urdf.xacro (robot description, xacro)
@@ -6,6 +6,9 @@
 	<xacro:include filename="$(find bot_description)/urdf/base/custom_base.gazebo.xacro" />
 	<!-- Wheel parameters -->
-	<xacro:property name="wheel_offset_x" value="0.2225" />    <!-- x,y,z in translation from base_link to the center of the wheel -->
-	<xacro:property name="wheel_offset_y" value="0.2045" />
+	<!-- <xacro:property name="wheel_offset_x" value="0.2225" />    x,y,z in translation from base_link to the center of the wheel -->
+	<!-- <xacro:property name="wheel_offset_y" value="0.2045" /> -->
+	<!-- <xacro:property name="wheel_offset_z" value="0.0" /> -->
+	<xacro:property name="wheel_offset_x" value="0.4450" />    <!-- x,y,z in translation from base_link to the center of the wheel -->
+	<xacro:property name="wheel_offset_y" value="0.4090" />
 	<xacro:property name="wheel_offset_z" value="0.0" />
 	<xacro:macro name="robot">

File: src/bot_description/urdf/wheels/omni_wheel.urdf.xacro (robot description, xacro)
@@ -20,10 +20,10 @@
         <xacro:if value="${reflect}">
           <geometry>
-            <mesh filename="package://bot_description/meshes/wheel/omni_wheel_1.dae" />
+            <mesh filename="package://bot_description/meshes/wheel/omni_wheel_1_scaled.dae" />
           </geometry>
           </xacro:if>
           <xacro:unless value="${reflect}">
             <geometry>
-              <mesh filename="package://bot_description/meshes/wheel/omni_wheel_2.dae" />
+              <mesh filename="package://bot_description/meshes/wheel/omni_wheel_2_scaled.dae" />
             </geometry>
 		    </xacro:unless>

File: src/bot_gazebo/urdf/camera.xacro (robot description, xacro)
@@ -47,6 +47,6 @@
                 <image>
                     <format>R8G8B8</format>
-                    <width>640</width>
-                    <height>640</height>
+                    <width>500</width>
+                    <height>500</height>
                 </image>
                 <clip>
