Commit message: daily commit

File: src/bot_description/urdf/tags/apriltag_demo.xacro (robot description, xacro)
@@ -4,6 +4,6 @@
   <xacro:include filename="$(find bot_description)/urdf/tags/apriltag_marker.xacro" />
   <link name="world"/>
-  <xacro:apriltag_marker namespace="" name="apriltag0" parent="world" family="36_11" ID="0" size="0.5">
-    <origin xyz="0 0 1" rpy=" 0 0 0" />
+  <xacro:apriltag_marker namespace="" name="apriltag0" parent="world" family="36h11" ID="0" size="0.5" apriltag_size="0.5">
+    <origin xyz="0 0 0" rpy=" 0 0 0" />
   </xacro:apriltag_marker>
 </robot>
