Commit message: daily commit

File: src/bot_description/urdf/full/bot.urdf.xacro (robot description, xacro)
@@ -28,4 +28,8 @@
 		<xacro:omni_steering />
    </xacro:macro>
+   <xacro:include filename="$(find bot_description)/urdf/tags/apriltag_marker.xacro" />
+   <xacro:apriltag_marker namespace="" name="apriltag0" parent="base_link" family="36h11" ID="0" size="0.5">
+    <origin xyz="0.1 0 0.65" rpy=" 0 0 0" />
+   </xacro:apriltag_marker>
    <xacro:robot/>
 </robot>

File: src/bot_gazebo/urdf/camera.xacro (robot description, xacro)
@@ -4,5 +4,5 @@
         <parent link="world"/>
         <child link="camera_link"/>
-        <origin xyz="0 0 5" rpy="0 0 0"/>
+        <origin xyz="0 0 5" rpy="0 1.57 0"/>
     </joint>
     <link name="world"/>
@@ -34,5 +34,6 @@
         <parent link="camera_link"/>
         <child link="camera_link_optical"/>
-        <origin xyz="0 0 0" rpy="${-pi/2} 0 ${-pi/2}"/>
+        <!-- <origin xyz="0 0 0" rpy="${-pi/2} 0 ${-pi/2}"/> -->
+        <origin xyz="0 0 0" rpy="0 0 0"/>
     </joint>
     <link name="camera_link_optical"></link>
@@ -40,5 +41,5 @@
         <material>Gazebo/Red</material>
         <sensor name="camera" type="camera">
-            <pose> 0 0 0 0 1.57 0 </pose>
+            <pose> 0 0 0 1.57 3.14 3.14 </pose>
             <visualize>true</visualize>
             <update_rate>30</update_rate>

Commit message: Added autonomous navigation packages and config. And odom from apriltag is developed
odom from tag yaw value is not good to use in realtime.So the imu odom
angle has to be used in custom costmap_plugin.And the ekf for imu odom
and tag odoms x,y has to be created.

File: src/bot_description/urdf/full/bot.urdf.xacro (robot description, xacro)
@@ -30,5 +30,5 @@
    <xacro:include filename="$(find bot_description)/urdf/tags/apriltag_marker.xacro" />
    <xacro:apriltag_marker namespace="" name="apriltag0" parent="base_link" family="36h11" ID="0" size="0.5">
-    <origin xyz="0.1 0 0.65" rpy=" 0 0 0" />
+    <origin xyz="0.0 0 0.625" rpy=" 0 0 0" />
    </xacro:apriltag_marker>
    <xacro:robot/>

Commit message: package holding platform for bot is added and package spawner file is added . both are in testing.

File: src/bot_description/urdf/full/bot.urdf.xacro (robot description, xacro)
@@ -33,3 +33,37 @@
    </xacro:apriltag_marker>
    <xacro:robot/>
+   <link name="package_platform">
+		<inertial>
+		<mass value="0.1" />
+		<origin xyz="0 0 0" rpy="0 0 1.5717"/>
+		<inertia  ixx="0.1" ixy="0.0"  ixz="0.0"  iyy="0.1"  iyz="0.0"  izz="0.1" />
+		</inertial>
+		<visual>
+		    <origin xyz="0 0.2 0" rpy="0 0 1.5717" />
+			<geometry>
+			<box size="0.25 0.5 0.05" />
+			</geometry>
+		</visual>
+	</link>
+	<joint name="package_platform_joint" type="revolute">
+		  <origin xyz="0.7 0 0.625" rpy="0 0 1.5717" />
+		  <parent link="base_link"/>
+		  <child link="package_platform" />
+		  <limit effort="15.0" lower="-1.57" upper="1.57" velocity="1"/>
+	</joint>
+	<transmission name="platform">
+    <type>transmission_interface/SimpleTransmission</type>
+    <joint name="package_platform_joint">
+      <hardwareInterface>hardware_interface/PositionJointInterface</hardwareInterface>
+    </joint>
+    <actuator name="package_platform_motor">
+      <hardwareInterface>hardware_interface/PositionJointInterface</hardwareInterface>
+      <mechanicalReduction>1</mechanicalReduction>
+    </actuator>
+  </transmission>
+  <gazebo>
+  <plugin name="gazebo_ros_control" filename="libgazebo_ros_control.so">
+    <robotNamespace>/</robotNamespace>
+  </plugin>
+</gazebo>
 </robot>

Commit message: package spawner updated and tested

File: src/bot_description/urdf/full/bot.urdf.xacro (robot description, xacro)
@@ -36,9 +36,15 @@
 		<inertial>
 		<mass value="0.1" />
-		<origin xyz="0 0 0" rpy="0 0 1.5717"/>
+		<origin xyz="0 0.1 0" rpy="0 0 1.5717"/>
 		<inertia  ixx="0.1" ixy="0.0"  ixz="0.0"  iyy="0.1"  iyz="0.0"  izz="0.1" />
 		</inertial>
+		<collision>
+       <origin xyz="0 0.15 0" rpy="0 0 0" />
+			<geometry>
+				<box size="0.25 0.5 0.05" />
+			</geometry>
+    	</collision>
 		<visual>
-		    <origin xyz="0 0.2 0" rpy="0 0 1.5717" />
+		    <origin xyz="0.0 0.15 0" rpy="0 0 1.5717" />
 			<geometry>
 			<box size="0.25 0.5 0.05" />
@@ -47,8 +53,8 @@
 	</link>
 	<joint name="package_platform_joint" type="revolute">
-		  <origin xyz="0.7 0 0.625" rpy="0 0 1.5717" />
+		  <origin xyz="0.85 0 0.625" rpy="0 0 1.5717" />
 		  <parent link="base_link"/>
 		  <child link="package_platform" />
-		  <limit effort="15.0" lower="-1.57" upper="1.57" velocity="1"/>
+		  <limit effort="50.0" lower="-1.57" upper="1.57" velocity="100"/>
 	</joint>
 	<transmission name="platform">

File: src/bot_package_manager/urdf/box.urdf (robot description, URDF)
Before this commit: robot package_red, 1 links, 0 joints
Links:
- link package: mass 0.02 -> 0.05; geometry collision box size=0.2 0.2 0.2; visual box size=0.2 0.2 0.2
